File: Untitled/Untitled.kicad_sch (KiCad schematic)
At the start: 77 parts, among them IC1 DRV8210, IC2 TPS7A2033, J1 5v in, J10 PROG, J11 Conn_01x08_Socket, J2 Volume, J3 Input, J4 IR, J5 Motor out, J6 Relays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

Commit message: MCP120-300 additiob
Parts:
- added R39: 10K, Resistor_SMD:R_0805_2012Metric_Pad1.20x1.40mm_HandSolder, symbol Device:R
- added U11: MCP120, Package_TO_SOT_SMD:SOT-23, symbol Power_Supervisor:MCP120-xxxxTT
- U4: value MCP23008-xSS -> MCP23008
Connections:
- net 3V3: now also R39.2, U11.2 (VDD)
- net GND: now also U11.3 (VSS)
- net PROG: now also R39.1, U11.1 (~{RST})
- net at U4.12 (GP0): now also R35.1; no longer R38.1
- net at U4.13 (GP1): now also R36.1; no longer R37.1
- net at U4.14 (GP2): now also R37.1; no longer R36.1
- net at U4.15 (GP3): now also R38.1; no longer R35.1
Other:
- moved on the sheet: J11, R31, R32, R33, R34, R35, R36, R37, R38
